File: fume Extractor.kicad_sch (KiCad schematic)
At the start: 11 parts, among them J1 FAN, Q1 BC337, SW1 SW_SPST, U1 L7805ACV

Commit message: fix: adjust pp cap and sizes
Parts:
- C1: footprint Capacitor_THT:C_Disc_D3.0mm_W2.0mm_P2.50mm -> Capacitor_THT:C_Rect_L10.0mm_W4.0mm_P7.50mm_MKS4
Changed lines of the file:
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@@
 			)
 		)
-		(property "Footprint" "Capacitor_THT:C_Disc_D3.0mm_W2.0mm_P2.50mm"
+		(property "Footprint" "Capacitor_THT:C_Rect_L10.0mm_W4.0mm_P7.50mm_MKS4"
 			(at 154.94 86.36 0)
 			(hide yes)

Commit message: feat: v2 with trimmer pot
Added RV2 to avoid long dead zones in RV1 because 500ohm is too much to
limit the 2V needed to minimally drive the fan, so the pot is largelly
dead. Adding a 1k 3266 Trimmer increases the ground resistance and the
floor voltage so we need to turn RV1 less to start the fan.

Plus, this gives a finer control over the fan speed itself
Parts:
- removed R2: 2R2k, Resistor_THT:R_Axial_DIN0207_L6.3mm_D2.5mm_P10.16mm_Horizontal, symbol PCM_SL_Devices:Resistor
- added RV2: 1K, Potentiometer_THT:Potentiometer_Bourns_3266W_Vertical, symbol Device:R_Potentiometer_Trim
- RV1: value 1K -> 500R
Connections:
- net -BATT: now also RV2.3
- net at C2.2, Q1.1 (C), RV1.1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: now also RV2.1
- net at RV1.3: now also RV2.2
Other:
- note added: "Adjust the trim (RV2) pot until the dead zone of RV1 is correct. If you don't, RV1 will have a super large dead zone"
- moved on the sheet: BT1

Commit message: Add Version 2
Parts:
- BT1: footprint Connector_Wire:SolderWire-0.127sqmm_1x02_P3.7mm_D0.48mm_OD1mm -> Connector_Molex:Molex_KK-254_AE-6410-02A_1x02_P2.54mm_Vertical
- D1: value LED_5mm -> LED_3mm; footprint LED_THT:LED_D5.0mm -> LED_THT:LED_D3.0mm
- RV1: footprint Potentiometer_THT:Potentiometer_Alpha_RD901F-40-00D_Single_Vertical -> Connector_Wire:SolderWire-0.5sqmm_1x03_P4.6mm_D0.9mm_OD2.1mm
- SW1: footprint User_Passives:SW_SPDT_100SP1T1B4M2QE -> PCM_4ms_Switch:Switch_Toggle_SPDT_SubMini
Connections:
- net at C2.2, Q1.1 (C), RV2.1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: now also RV1.3; no longer RV1.1
- net at RV2.2: now also RV1.1; no longer RV1.3
- net at C1.1, R1.2, U1.1 (IN): now also SW1.1; no longer SW1.3
Other:
- moved on the sheet: RV1
Changed lines of the file:
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@@
+	)
+	(junction
+		(at 191.77 77.47)
+		(diameter 0)
+		(color 0 0 0 0)
 	)
 	(junction
@@
 	)
 	(junction
-		(at 190.5 77.47)
+		(at 151.13 71.12)
 		(diameter 0)
 		(color 0 0 0 0)
 	)
 	(junction
-		(at 151.13 71.12)
+		(at 127 76.2)
+		(diameter 0)
+		(color 0 0 0 0)
+	)
+	(junction
+		(at 127 68.58)
+		(diameter 0)
+		(color 0 0 0 0)
+	)
+	(junction
+		(at 153.67 71.12)
 		(diameter 0)
 		(color 0 0 0 0)
@@
 		(color 0 0 0 0)
 	)
-	(junction
-		(at 127 76.2)
-		(diameter 0)
-		(color 0 0 0 0)
-	)
-	(junction
-		(at 127 68.58)
-		(diameter 0)
-		(color 0 0 0 0)
-	)
-	(junction
-		(at 153.67 71.12)
-		(diameter 0)
-		(color 0 0 0 0)
-	)
 	(no_connect
 		(at 151.13 66.04)
@@
 	(wire
 		(pts
-			(xy 190.5 77.47) (xy 190.5 71.12)
+			(xy 191.77 77.47) (xy 191.77 71.12)
 		)
 		(stroke
@@
 	(wire
 		(pts
-			(xy 179.07 71.12) (xy 190.5 71.12)
+			(xy 179.07 71.12) (xy 191.77 71.12)
 		)
 		(stroke
@@
 			)
 		)
-		(property "Value" "LED_5mm"
+		(property "Value" "LED_3mm"
 			(at 142.494 85.852 0)
 			(hide yes)
@@
 			)
 		)
-		(property "Footprint" "LED_THT:LED_D5.0mm"
+		(property "Footprint" "LED_THT:LED_D3.0mm"
 			(at 145.796 79.756 0)
 			(hide yes)
@@
 		)
 		(instances
-			(project "kicadrt_analysis_fume Extractor"
+			(project "fume Extractor"
 				(path "/d6602a71-2883-441a-8964-9fddcde39fdc"
 					(reference "D1")
@@
 	(symbol
 		(lib_id "Device:R_Potentiometer")
-		(at 186.69 77.47 270)
+		(at 186.69 77.47 90)
+		(mirror x)
 		(unit 1)
 		(body_style 1)
@@
 		(dnp no)
 		(property "Reference" "RV1"
-			(at 186.436 73.152 90)
+			(at 186.944 73.152 90)
 			(show_name no)
 			(do_not_autoplace no)
@@
 			)
 		)
-		(property "Footprint" "Potentiometer_THT:Potentiometer_Alpha_RD901F-40-00D_Single_Vertical"
+		(property "Footprint" "Connector_Wire:SolderWire-0.5sqmm_1x03_P4.6mm_D0.9mm_OD2.1mm"
 			(at 186.69 77.47 0)
 			(hide yes)
@@
 		)
 		(instances
-			(project "kicadrt_analysis_fume Extractor"
+			(project "fume Extractor"
 				(path "/d6602a71-2883-441a-8964-9fddcde39fdc"
 					(reference "RV1")
@@
 		)
 		(instances
-			(project "kicadrt_analysis_fume Extractor"
+			(project "fume Extractor"
 				(path "/d6602a71-2883-441a-8964-9fddcde39fdc"
 					(reference "C1")
@@
 		)
 		(instances
-			(project "kicadrt_analysis_fume Extractor"
+			(project "fume Extractor"
 				(path "/d6602a71-2883-441a-8964-9fddcde39fdc"
 					(reference "#PWR01")
@@
 		(lib_id "User_Passives:100SP1T1B4M2QE")
 		(at 143.51 68.58 0)
+		(mirror x)
 		(unit 1)
 		(body_style 1)
@@
 		(in_pos_files yes)
 		(dnp no)
-		(fields_autoplaced yes)
 		(property "Reference" "SW1"
-			(at 143.51 63.5 0)
+			(at 143.51 73.66 0)
 			(show_name no)
 			(do_not_autoplace no)
@@
 		)
 		(property "Value" "SW_SPST"
-			(at 143.51 64.77 0)
-			(hide yes)
-			(show_name no)
-			(do_not_autoplace no)
-			(effects
-				(font
-					(size 1.27 1.27)
-				)
-			)
-		)
-		(property "Footprint" "User_Passives:SW_SPDT_100SP1T1B4M2QE"
+			(at 143.51 72.39 0)
+			(hide yes)
+			(show_name no)
+			(do_not_autoplace no)
+			(effects
+				(font
+					(size 1.27 1.27)
+				)
+			)
+		)
+		(property "Footprint" "PCM_4ms_Switch:Switch_Toggle_SPDT_SubMini"
 			(at 143.51 68.58 0)
 			(hide yes)
@@
 		)
 		(instances
-			(project "kicadrt_analysis_fume Extractor"
+			(project "fume Extractor"
 				(path "/d6602a71-2883-441a-8964-9fddcde39fdc"
 					(reference "SW1")
@@
 			)
 		)
-		(property "Footprint" "Connector_Wire:SolderWire-0.127sqmm_1x02_P3.7mm_D0.48mm_OD1mm"
+		(property "Footprint" "Connector_Molex:Molex_KK-254_AE-6410-02A_1x02_P2.54mm_Vertical"
 			(at 127 72.136 90)
 			(hide yes)
@@
 		)
 		(instances
-			(project "kicadrt_analysis_fume Extractor"
+			(project "fume Extractor"
 				(path "/d6602a71-2883-441a-8964-9fddcde39fdc"
 					(reference "BT1")
@@
 		)
 		(instances
-			(project "kicadrt_analysis_fume Extractor"
+			(project "fume Extractor"
 				(path "/d6602a71-2883-441a-8964-9fddcde39fdc"
 					(reference "#FLG04")
@@
 		)
 		(instances
-			(project "kicadrt_analysis_fume Extractor"
+			(project "fume Extractor"
 				(path "/d6602a71-2883-441a-8964-9fddcde39fdc"
 					(reference "#FLG01")
@@
 		)
 		(instances
-			(project "kicadrt_analysis_fume Extractor"
+			(project "fume Extractor"
 				(path "/d6602a71-2883-441a-8964-9fddcde39fdc"
 					(reference "U1")
@@
 		)
 		(instances
-			(project "kicadrt_analysis_fume Extractor"
+			(project "fume Extractor"
 				(path "/d6602a71-2883-441a-8964-9fddcde39fdc"
 					(reference "J1")
@@
 		)
 		(instances
-			(project "kicadrt_analysis_fume Extractor"
+			(project "fume Extractor"
 				(path "/d6602a71-2883-441a-8964-9fddcde39fdc"
 					(reference "RV2")
@@
 		)
 		(instances
-			(project "kicadrt_analysis_fume Extractor"
+			(project "fume Extractor"
 				(path "/d6602a71-2883-441a-8964-9fddcde39fdc"
 					(reference "#PWR02")
@@
 		)
 		(instances
-			(project "kicadrt_analysis_fume Extractor"
+			(project "fume Extractor"
 				(path "/d6602a71-2883-441a-8964-9fddcde39fdc"
 					(reference "C2")
@@
 		)
 		(instances
-			(project "kicadrt_analysis_fume Extractor"
+			(project "fume Extractor"
 				(path "/d6602a71-2883-441a-8964-9fddcde39fdc"
 					(reference "#FLG03")
@@
 		)
 		(instances
-			(project "kicadrt_analysis_fume Extractor"
+			(project "fume Extractor"
 				(path "/d6602a71-2883-441a-8964-9fddcde39fdc"
 					(reference "R1")
@@
 		)
 		(instances
-			(project "kicadrt_analysis_fume Extractor"
+			(project "fume Extractor"
 				(path "/d6602a71-2883-441a-8964-9fddcde39fdc"
 					(reference "Q1")
